File: fluidics-v2/uartshift.kicad_sch (KiCad schematic)
At the start: 5 parts, among them IC2 PI4ULS5V202UEX

Commit message: new version
Parts:
- IC2: footprint MAX232:SOP65P640X120-16N -> uart_lvlshift:SOP65P490X110-8N
Other:
- note added: "find IC that lists uart as an application"
Changed lines of the file:
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@@
     (stroke (width 0) (type default))
+  )
+  (text "find IC that lists uart as an application\n" (at 111.76 87.63 0)
+    (effects (font (size 1.27 1.27)) (justify left bottom))
   )
   (hierarchical_label "RX_3.3" (shape input) (at 110.49 73.66 180) (fields_autoplaced)
@@
       (effects (font (size 1.27 1.27)))
     )
-    (property "Footprint" "MAX232:SOP65P640X120-16N" (at 134.62 166.04 0)
+    (property "Footprint" "uart_lvlshift:SOP65P490X110-8N" (at 134.62 166.04 0)
       (effects (font (size 1.27 1.27)) (justify left top) hide)
     )
